File: Shard.kicad_sch (KiCad schematic)
At the start: 52 parts, among them J1 USB_C_Receptacle_USB2.0_16P, J2 Conn_01x08, J3 Conn_01x08, J4 Conn_01x08, J5 Conn_01x08, SW1 SW_Push, SW2 SW_Push, U1 ESP32-S3, U2 USBLC6-2P6, U3 TLV76733DRVx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

Commit message: USB-C PCB routing
Parts:
- C17, C18: footprint (none) -> Capacitor_SMD:C_0201_0603Metric; REF (none) -> C426053
- J2, J3, J4, J5: footprint (none) -> Connector_PinSocket_2.54mm:PinSocket_1x08_P2.54mm_Vertical
Connections:
- net GND: now also J5.5 (Pin_5)
- net RESET: now also J5.2 (Pin_2); no longer J5.3 (Pin_3)
- net RX: now also J5.3 (Pin_3); no longer J5.4 (Pin_4)
- net TX: now also J5.4 (Pin_4); no longer J5.5 (Pin_5)
- net at D2.2 (A): now also J5.1 (Pin_1); no longer J5.2 (Pin_2)
- net D_P: now reaches J1.A6 (D+), J1.B6 (D+), U2.3 (I/O2)
- net D_N: now reaches J1.A7 (D-), J1.B7 (D-), U2.1 (I/O1)
- net SPICS1: no longer names the net of U1.28 (SPICS1)
Other:
- moved on the sheet: D2
Changed lines of the file:
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@@
 	)
 	(junction
+		(at 77.47 123.19)
+		(diameter 0)
+		(color 0 0 0 0)
+	)
+	(junction
 		(at 25.4 151.13)
 		(diameter 0)
@@
 	)
 	(no_connect
-		(at 76.2 135.89)
-	)
-	(no_connect
 		(at 195.58 80.01)
 	)
@@
 	)
 	(no_connect
+		(at 195.58 36.83)
+	)
+	(no_connect
 		(at 195.58 59.69)
 	)
@@
 	(wire
 		(pts
+			(xy 77.47 123.19) (xy 77.47 125.73)
+		)
+		(stroke
+			(width 0)
+			(type default)
+		)
+	)
+	(wire
+		(pts
 			(xy 144.78 57.15) (xy 149.86 57.15)
 		)
@@
 	(wire
 		(pts
+			(xy 83.82 135.89) (xy 85.09 135.89)
+		)
+		(stroke
+			(width 0)
+			(type default)
+		)
+	)
+	(wire
+		(pts
 			(xy 49.53 82.55) (xy 55.88 82.55)
 		)
@@
 	(wire
 		(pts
+			(xy 77.47 125.73) (xy 76.2 125.73)
+		)
+		(stroke
+			(width 0)
+			(type default)
+		)
+	)
+	(wire
+		(pts
 			(xy 256.54 81.28) (xy 256.54 91.44)
 		)
@@
 	(wire
 		(pts
-			(xy 195.58 36.83) (xy 212.09 36.83)
-		)
-		(stroke
-			(width 0)
-			(type default)
-		)
-	)
-	(wire
-		(pts
 			(xy 256.54 91.44) (xy 250.19 91.44)
 		)
@@
 		)
 	)
+	(label "D_P"
+		(at 50.8 85.09 0)
+		(fields_autoplaced yes)
+		(effects
+			(font
+				(size 1.27 1.27)
+			)
+			(justify left bottom)
+		)
+	)
 	(label "2"
 		(at 144.78 41.91 180)
@@
 	)
 	(label "RESET"
-		(at 76.2 130.81 0)
+		(at 76.2 133.35 0)
 		(fields_autoplaced yes)
 		(effects
@@
 	)
 	(label "RX"
-		(at 76.2 128.27 0)
+		(at 76.2 130.81 0)
 		(fields_autoplaced yes)
 		(effects
@@
 		)
 	)
-	(label "D+"
-		(at 72.39 85.09 0)
+	(label "D_N"
+		(at 50.8 82.55 0)
 		(fields_autoplaced yes)
 		(effects
@@
 		)
 	)
-	(label "SPICS1"
-		(at 212.09 36.83 0)
+	(label "D+"
+		(at 72.39 85.09 0)
 		(fields_autoplaced yes)
 		(effects
@@
 	)
 	(label "TX"
-		(at 76.2 125.73 0)
+		(at 76.2 128.27 0)
 		(fields_autoplaced yes)
 		(effects
@@
 	)
 	(label "VIN"
-		(at 83.82 133.35 0)
+		(at 85.09 135.89 0)
 		(fields_autoplaced yes)
 		(effects
@@
 			)
 		)
-		(property "Footprint" ""
+		(property "Footprint" "Connector_PinSocket_2.54mm:PinSocket_1x08_P2.54mm_Vertical"
 			(at 38.1 128.27 0)
 			(effects
@@
 	(symbol
 		(lib_id "Device:D_Schottky")
-		(at 80.01 133.35 180)
+		(at 80.01 135.89 180)
 		(unit 1)
 		(exclude_from_sim no)
@@
 		(dnp no)
 		(property "Reference" "D2"
-			(at 80.01 135.89 0)
+			(at 80.01 138.43 0)
 			(effects
 				(font
@@
 		)
 		(property "Value" "SS34"
-			(at 86.106 135.382 0)
+			(at 86.106 137.922 0)
 			(effects
 				(font
@@
 		)
 		(property "Footprint" "Diode_SMD:D_SMA"
-			(at 80.01 133.35 0)
+			(at 80.01 135.89 0)
 			(effects
 				(font
@@
 		)
 		(property "Datasheet" "~"
-			(at 80.01 133.35 0)
+			(at 80.01 135.89 0)
 			(effects
 				(font
@@
 		)
 		(property "Description" "Schottky diode"
-			(at 80.01 133.35 0)
+			(at 80.01 135.89 0)
 			(effects
 				(font
@@
 		)
 		(property "REF" "C8678"
-			(at 80.01 133.35 0)
+			(at 80.01 135.89 0)
 			(effects
 				(font
@@
 			)
 		)
-		(property "Footprint" ""
+		(property "Footprint" "Connector_PinSocket_2.54mm:PinSocket_1x08_P2.54mm_Vertical"
 			(at 29.21 125.73 0)
 			(effects
@@
 			)
 		)
-		(property "Footprint" ""
+		(property "Footprint" "Connector_PinSocket_2.54mm:PinSocket_1x08_P2.54mm_Vertical"
 			(at 71.12 128.27 0)
 			(effects
@@
 			)
 		)
-		(property "Footprint" ""
+		(property "Footprint" "Capacitor_SMD:C_0201_0603Metric"
 			(at 263.8552 87.63 0)
 			(effects
@@
 			)
 		)
+		(property "REF" " C426053"
+			(at 262.89 83.82 0)
+			(effects
+				(font
+					(size 1.27 1.27)
+				)
+				(hide yes)
+			)
+		)
 		(pin "2"
 		)
@@
 			)
 		)
-		(property "Footprint" ""
+		(property "Footprint" "Capacitor_SMD:C_0201_0603Metric"
 			(at 251.1552 87.63 0)
 			(effects
@@
 			)
 		)
+		(property "REF" " C426053"
+			(at 250.19 83.82 0)
+			(effects
+				(font
+					(size 1.27 1.27)
+				)
+				(hide yes)
+			)
+		)
 		(pin "2"
 		)
@@
 			)
 		)
-		(property "Footprint" ""
+		(property "Footprint" "Connector_PinSocket_2.54mm:PinSocket_1x08_P2.54mm_Vertical"
 			(at 62.23 125.73 0)
 			(effects

Commit message: Finish initial PCB Layout
Parts:
- ANT1: footprint RF_Antenna:Texas_SWRA117D_2.4GHz_Left -> RF_Antenna:Texas_SWRA117D_2.4GHz_Right
- C1, C13, C15, C3, C6, C9: footprint Capacitor_SMD:C_0603_1608Metric -> Capacitor_SMD:C_0201_0603Metric; REF C106214 -> C5209398
- C10, C11, C12, C16, C7, C8: footprint Capacitor_SMD:C_1206_3216Metric -> Capacitor_SMD:C_0201_0603Metric; REF C93194 -> C312124
- C4: footprint Capacitor_SMD:C_1206_3216Metric -> Capacitor_SMD:C_0201_0603Metric; REF C77500 -> C312126
- R11: footprint Resistor_SMD:R_0805_2012Metric -> Resistor_SMD:R_0201_0603Metric; REF C2933536 -> C306975
Changed lines of the file:
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@@
 			)
 		)
-		(property "Footprint" "Capacitor_SMD:C_0603_1608Metric"
+		(property "Footprint" "Capacitor_SMD:C_0201_0603Metric"
 			(at 91.1352 33.02 0)
 			(effects
@@
 			)
 		)
-		(property "REF" " C106214"
+		(property "REF" " C5209398"
 			(at 90.17 29.21 0)
 			(effects
@@
 			)
 		)
-		(property "Footprint" "Capacitor_SMD:C_1206_3216Metric"
+		(property "Footprint" "Capacitor_SMD:C_0201_0603Metric"
 			(at 61.9252 184.15 0)
 			(effects
@@
 			)
 		)
-		(property "REF" "C93194"
+		(property "REF" " C312124"
 			(at 60.96 180.34 0)
 			(effects
@@
 			)
 		)
-		(property "Footprint" "Capacitor_SMD:C_0603_1608Metric"
+		(property "Footprint" "Capacitor_SMD:C_0201_0603Metric"
 			(at 75.8952 160.02 0)
 			(effects
@@
 			)
 		)
-		(property "REF" " C106214"
+		(property "REF" " C5209398"
 			(at 74.93 156.21 0)
 			(effects
@@
 			)
 		)
-		(property "Footprint" "Capacitor_SMD:C_1206_3216Metric"
+		(property "Footprint" "Capacitor_SMD:C_0201_0603Metric"
 			(at 87.3252 160.02 0)
 			(effects
@@
 			)
 		)
-		(property "REF" "C93194"
+		(property "REF" " C312124"
 			(at 86.36 156.21 0)
 			(effects
@@
 			)
 		)
-		(property "Footprint" "Capacitor_SMD:C_1206_3216Metric"
+		(property "Footprint" "Capacitor_SMD:C_0201_0603Metric"
 			(at 40.3352 160.02 0)
 			(effects
@@
 			)
 		)
-		(property "REF" "C77500"
+		(property "REF" " C312126"
 			(at 39.37 156.21 0)
 			(effects
@@
 			)
 		)
-		(property "Footprint" "Capacitor_SMD:C_0603_1608Metric"
+		(property "Footprint" "Capacitor_SMD:C_0201_0603Metric"
 			(at 26.3652 160.02 0)
 			(effects
@@
 			)
 		)
-		(property "REF" " C106214"
+		(property "REF" " C5209398"
 			(at 25.4 156.21 0)
 			(effects
@@
 			)
 		)
-		(property "Footprint" "Capacitor_SMD:C_1206_3216Metric"
+		(property "Footprint" "Capacitor_SMD:C_0201_0603Metric"
 			(at 39.0652 184.15 0)
 			(effects
@@
 			)
 		)
-		(property "REF" "C93194"
+		(property "REF" " C312124"
 			(at 38.1 180.34 0)
 			(effects
@@
 			)
 		)
-		(property "Footprint" "Capacitor_SMD:C_0603_1608Metric"
+		(property "Footprint" "Capacitor_SMD:C_0201_0603Metric"
 			(at 26.3652 184.15 0)
 			(effects
@@
 			)
 		)
-		(property "REF" " C106214"
+		(property "REF" " C5209398"
 			(at 25.4 180.34 0)
 			(effects
@@
 			)
 		)
-		(property "Footprint" "Capacitor_SMD:C_0603_1608Metric"
+		(property "Footprint" "Capacitor_SMD:C_0201_0603Metric"
 			(at 145.7452 168.91 0)
 			(effects
@@
 			)
 		)
-		(property "REF" " C106214"
+		(property "REF" " C5209398"
 			(at 144.78 165.1 0)
 			(effects
@@
 			)
 		)
-		(property "Footprint" "Capacitor_SMD:C_1206_3216Metric"
+		(property "Footprint" "Capacitor_SMD:C_0201_0603Metric"
 			(at 102.5652 160.02 0)
 			(effects
@@
 			)
 		)
-		(property "REF" "C93194"
+		(property "REF" " C312124"
 			(at 101.6 156.21 0)
 			(effects
@@
 			)
 		)
-		(property "Footprint" "Capacitor_SMD:C_1206_3216Metric"
+		(property "Footprint" "Capacitor_SMD:C_0201_0603Metric"
 			(at 267.6652 132.08 0)
 			(effects
@@
 			)
 		)
-		(property "REF" "C93194"
+		(property "REF" " C312124"
 			(at 266.7 128.27 0)
 			(effects
@@
 			)
 		)
-		(property "Footprint" "Resistor_SMD:R_0805_2012Metric"
+		(property "Footprint" "Resistor_SMD:R_0201_0603Metric"
 			(at 241.3 80.518 90)
 			(effects
@@
 			)
 		)
-		(property "REF" " C2933536"
+		(property "REF" "C306975"
 			(at 241.3 78.74 90)
 			(effects
@@
 			)
 		)
-		(property "Footprint" "Capacitor_SMD:C_1206_3216Metric"
+		(property "Footprint" "Capacitor_SMD:C_0201_0603Metric"
 			(at 87.3252 184.15 0)
 			(effects
@@
 			)
 		)
-		(property "REF" "C93194"
+		(property "REF" " C312124"
 			(at 86.36 180.34 0)
 			(effects
@@
 			)
 		)
-		(property "Footprint" "Capacitor_SMD:C_0603_1608Metric"
+		(property "Footprint" "Capacitor_SMD:C_0201_0603Metric"
 			(at 27.6352 33.02 0)
 			(effects
@@
 			)
 		)
-		(property "REF" " C106214"
+		(property "REF" " C5209398"
 			(at 26.67 29.21 0)
 			(effects
@@
 			)
 		)
-		(property "Footprint" "RF_Antenna:Texas_SWRA117D_2.4GHz_Left"
+		(property "Footprint" "RF_Antenna:Texas_SWRA117D_2.4GHz_Right"
 			(at 229.87 34.29 0)
 			(effects
